File: Hardware/SparkFun_Qwiic_CO2_Sensor_STCC4.kicad_sch (KiCad schematic)
At the start: 27 parts, among them J1 Qwiic_RA, J2 Qwiic_RA, J3 Conn_01x06, U2 STCC4, U3 SHT40

Commit message: Added changes from Design Review
- Nudged vias
- Replaced "pullup" capacitors
- Adjusted measures alignment
- Adjusted solder paste expansion
- Swapped Flame and OSHW Logos
Parts:
- R4, R5: value 0.1uF -> 2.2k; footprint SparkFun-Capacitor:C_0603_1608Metric -> SparkFun-Resistor:R_0603_1608Metric; symbol SparkFun-Capacitor:0.1uF_0603_25V_20% -> SparkFun-Resistor:2.2k_0603; PROD_ID CAP-00810 -> RES-08272; Tolerance 20% -> (none); Voltage 25V -> (none)
Connections:
- net SCL: now also R4.2; no longer R4.1
- net SDA: now also R5.2; no longer R5.1
- net at JP2.1 (A): now also R5.1; no longer R5.2
- net at JP2.3 (C): now also R4.1; no longer R4.2
Other:
- moved on the sheet: C10, C11, R4, R5, U2, U3
