File: Hardware/SparkFun_Qwiic_CO2_Sensor_STCC4.kicad_pcb (KiCad board)
At the start: 2 copper layers, 25.4 x 25.4 mm, 46 parts, among them J1 Qwiic_RA, J2 Qwiic_RA, J3 Conn_01x06, U2 STCC4, U3 SHT40

Commit message: Updated to v10 for REDs
Other:
- board text added: "v10"
- board text removed: "v01"
Changed lines of the file:
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@@
 		(title "SparkFun Qwiic CO2 Sensor STCC4")
 		(date "2026-05-15")
-		(rev "v01")
+		(rev "v10")
 		(company "SparkFun Electronics")
 		(comment 1 "Designed by: Geoff McIntyre")
@@
 		(layer "Edge.Cuts")
 	)
-	(gr_text "v01"
+	(gr_text "v10"
 		(at 125.171 92.391 270)
 		(layer "B.Cu" knockout)
@@
 			(keep_text_aligned yes)
 		)
-		(gr_text "0.9 in"
+		(gr_text "900 mils"
 			(at 115.4461 99.376 90)
 			(layer "Dwgs.User")
@@
 			(keep_text_aligned yes)
 		)
-		(gr_text "1 in"
+		(gr_text "1000 mils"
 			(at 113.2236 98.106 90)
 			(layer "Dwgs.User")
@@
 			(keep_text_aligned yes)
 		)
-		(gr_text "1 in"
+		(gr_text "1000 mils"
 			(at 135.966 119.1786 0)
 			(layer "Dwgs.User")
@@
 			(keep_text_aligned yes)
 		)
-		(gr_text "0.9 in"
+		(gr_text "900 mils"
 			(at 134.696 116.6386 0)
 			(layer "Dwgs.User")
@@
 			(extension_offset 0.5)
 		)
-		(gr_text "0.1 in"
+		(gr_text "100 mils"
 			(at 135.0135 113.981 0)
 			(layer "Dwgs.User")
@@
 			(extension_offset 0.5)
 		)
-		(gr_text "0.5 in"
+		(gr_text "500 mils"
 			(at 117.6686 104.456 90)
 			(layer "Dwgs.User")
@@
 			(keep_text_aligned yes)
 		)
-		(gr_text "0.1 in"
+		(gr_text "100 mils"
 			(at 121.6785 107.9485 90)
 			(layer "Dwgs.User")
@@
 			(keep_text_aligned yes)
 		)
-		(gr_text "0.35 in"
+		(gr_text "350 mils"
 			(at 131.267 115.886 0)
 			(layer "Dwgs.User")
